File: Eagle/Cass2SD.brd (EAGLE design)
At the start: 100 x 80 mm, 33 parts, among them IC1 MCP1702-5002, IC2 ATMEGA328P-PU, IC3 LM358N, Q1 8MHz, SW1 EC12E_SW, X1 MAB5SH

Commit message: Changed to external XTAL with 16MHz
Parts:
- C1: value 10µ -> 47µ
- C8: value 10µ -> 22µ
- R1: value 10k -> 12k
- R4: value 10k -> 27k
- R5: value 10k -> 5k
- R8: value 270 -> 330
